File: HamPWR.kicad_pcb (KiCad board)
At the start: 4 copper layers, 100 x 100 mm, 660 parts, among them J1 CTRL, J10 VDDP, J11 PHASE, J12 VFB, J13 VSYS, J2 VREF, J3 VC, J4 GND, J5 VIN, J6 VOUT, J7 ICREF, J8 FBO, J9 BOOT, Q1 2N7002P, Q2 2N7002P, Q3 2N7002P, Q4 DMP10H4D2S, U1 LT3790, U10 bq24765, U11 Si4435DY, U12 Si4435DY, U13 Si4435DY, U2 SQJ459EP, U3 SQJ459EP, U4 BSC032N04LS, U5 BSC032N04LS, U6 SQJ459EP, U7 SQJ459EP, U8 BSC032N04LS, U9 BSC032N04LS

Commit message: Progress
Parts:
- removed the REF** at (143.0, 121.8)
- removed the REF** at (137.8, 148.5)
- removed the REF** at (134.5, 148.5)
- removed the REF** at (58.0, 142.0)
- removed the REF** at (75.8, 56.1)
- removed the REF** at (54.2, 142.0)
- removed the REF** at (58.0, 146.8)
- removed the REF** at (54.2, 146.8)
- removed the REF** at (75.0, 58.9)
- removed the REF** at (72.8, 56.1)
- removed the REF** at (70.8, 53.4)
- removed the REF** at (67.5, 53.4)
- removed the REF** at (67.5, 56.9)
- removed the REF** at (70.3, 58.9)
- removed the REF** at (70.3, 62.9)
- removed the REF** at (67.5, 60.9)
- removed the REF** at (64.5, 58.9)
- removed the REF** at (64.5, 62.9)
- removed the REF** at (61.3, 60.9)
- removed the REF** at (58.0, 58.9)
- removed the REF** at (57.8, 62.9)
- removed the REF** at (55.0, 60.9)
- removed the REF** at (52.5, 58.9)
- removed the REF** at (52.5, 62.9)
- removed the REF** at (52.5, 66.1)
- removed the REF** at (52.5, 71.1)
- removed the REF** at (52.5, 76.6)
- removed the REF** at (52.5, 81.8)
- removed the REF** at (127.5, 147.2)
- removed the REF** at (130.0, 147.2)
- removed the REF** at (52.5, 87.1)
- removed the REF** at (123.0, 147.2)
- removed the REF** at (125.5, 147.2)
- removed the REF** at (52.5, 91.8)
- removed the REF** at (117.8, 147.2)
- removed the REF** at (120.2, 147.2)
- removed the REF** at (54.8, 94.6)
- removed the REF** at (112.8, 147.2)
- removed the REF** at (115.2, 147.2)
- removed the REF** at (107.8, 147.2)
- removed the REF** at (52.5, 96.1)
- removed the REF** at (110.2, 147.2)
- removed the REF** at (105.2, 147.2)
- removed the REF** at (54.8, 97.6)
- removed the REF** at (102.8, 147.2)
- removed the REF** at (68.5, 147.2)
- removed the REF** at (58.5, 94.6)
- removed the REF** at (73.2, 147.2)
- removed the REF** at (78.5, 147.2)
- removed the REF** at (56.8, 96.1)
- removed the REF** at (76.0, 147.2)
- removed the REF** at (58.5, 97.6)
- removed the REF** at (70.8, 147.2)
- removed the REF** at (81.2, 147.2)
- removed the REF** at (83.8, 147.2)
- removed the REF** at (89.0, 147.2)
- removed the REF** at (62.8, 97.6)
- removed the REF** at (86.5, 147.2)
- removed the REF** at (94.5, 147.2)
- removed the REF** at (61.0, 96.1)
- removed the REF** at (92.0, 147.2)
- removed the REF** at (99.8, 147.2)
- removed the REF** at (97.2, 147.2)
- removed the REF** at (62.8, 94.6)
- removed the REF** at (61.0, 92.8)
- removed the REF** at (62.8, 91.3)
- removed the REF** at (61.0, 89.8)
- removed the REF** at (62.8, 88.3)
- removed the REF** at (61.0, 87.1)
- removed the REF** at (62.0, 85.3)
- removed the REF** at (64.8, 81.3)
- removed the REF** at (63.8, 82.8)
- removed the REF** at (61.3, 83.8)
- added C54: 10µF 100V, Capacitors_SMD:C_1210, F.Cu at (134.8, 98.8)
- added C55: 10µF 100V, Capacitors_SMD:C_1210, F.Cu at (134.8, 95.5)
- added C56: 10µF 100V, Capacitors_SMD:C_1210, F.Cu at (125.5, 100.0)
- added C57: 10µF 100V, Capacitors_SMD:C_1210, F.Cu at (125.5, 96.8)
- added C58: 220µF 35V, Capacitors_SMD:CP_Elec_8x10.5, F.Cu at (58.8, 107.8)
- added C59: 20pF, Capacitors_SMD:C_0402, F.Cu at (127.5, 56.5)
- added C60: 20pF, Capacitors_SMD:C_0402, F.Cu at (127.2, 61.5)
- added C61: 10µF, Capacitors_SMD:C_0603, F.Cu at (127.2, 58.8)
- added C62: 100nF, Capacitors_SMD:C_0201, B.Cu at (121.0, 64.0)
- added C63: 100nF, Capacitors_SMD:C_0201, B.Cu at (120.0, 57.8)
- added C64: 39nF, Capacitors_SMD:C_0201, F.Cu at (130.2, 68.0)
- added C65: 22nF, Capacitors_SMD:C_0201, B.Cu at (112.4, 64.0)
- added C66: 10µF, Capacitors_SMD:C_0603, F.Cu at (121.5, 69.2)
- added C67: 100nF, Capacitors_SMD:C_0201, F.Cu at (112.0, 70.8)
- added C68: 3.3nF, Capacitors_SMD:C_0201, F.Cu at (118.2, 71.8)
- added C69: 10µF, Capacitors_SMD:C_0603, F.Cu at (100.2, 61.5)
- added C70: 100nF, Capacitors_SMD:C_0201, F.Cu at (105.0, 70.5)
- added C71: 22nF, Capacitors_SMD:C_0201, F.Cu at (103.2, 66.8)
- added C72: 10µF, Capacitors_SMD:C_0603, F.Cu at (106.0, 63.0)
- added C73: 100nF, Capacitors_SMD:C_0201, F.Cu at (100.5, 70.2)
- added C74: 100nF, Capacitors_SMD:C_0201, F.Cu at (106.7, 60.2)
- added D9: 10V, Diodes_SMD:D_SOD-123, F.Cu at (140.5, 97.8)
- added F1: 10A Fast, 0685H9100-01, Fuse_Holders_and_Fuses:Fuse_SMD1206_Reflow, F.Cu at (146.0, 98.0)
- added J14: PJ-082BH, stuff:pj-082bh, F.Cu at (135.8, 108.2)
- added L3: SRP1265A-5R6M, stuff:SRP1265A, F.Cu at (125.9, 108.0)
- added L4: BLM15HG601SN1D, Inductors_SMD:L_0402, F.Cu at (98.8, 65.0)
- added L5: BLM15HG601SN1D, Inductors_SMD:L_0402, F.Cu at (102.3, 57.2)
- added R71: 10k, Resistors_SMD:R_0402, F.Cu at (142.9, 96.0)
- added REF**: Via, stuff:Via, F.Cu at (121.2, 92.8)
- added REF**: Via, stuff:Via, F.Cu at (113.8, 87.8)
- added REF**: Via, stuff:Via, F.Cu at (129.8, 94.8)
- added REF**: Via, stuff:Via, F.Cu at (131.7, 92.3)
- added REF**: Via, stuff:Via, F.Cu at (129.3, 92.2)
- added REF**: Via, stuff:Via, F.Cu at (122.5, 96.5)
- added REF**: Via, stuff:Via, F.Cu at (122.5, 99.5)
- added REF**: Via, stuff:Via, F.Cu at (121.8, 102.2)
- added REF**: Via, stuff:Via, F.Cu at (118.0, 104.7)
- added REF**: Via, stuff:Via, F.Cu at (119.8, 104.0)
- added REF**: Via, stuff:Via, F.Cu at (121.8, 104.0)
- added REF**: Via, stuff:Via, F.Cu at (121.8, 106.0)
- added REF**: Via, stuff:Via, F.Cu at (118.8, 87.8)
- added REF**: Via, stuff:Via, F.Cu at (121.8, 108.0)
- added REF**: Via, stuff:Via, F.Cu at (121.8, 109.8)
- added REF**: Via, stuff:Via, F.Cu at (137.9, 100.2)
- added REF**: Via, stuff:Via, F.Cu at (132.3, 110.3)
- added REF**: Via, stuff:Via, F.Cu at (134.6, 109.8)
- added REF**: Via, stuff:Via, F.Cu at (134.6, 106.5)
- added REF**: Via, stuff:Via, F.Cu at (134.6, 104.5)
- added REF**: Via, stuff:Via, F.Cu at (132.3, 104.5)
- added REF**: Via, stuff:Via, F.Cu at (133.9, 102.8)
- added REF**: Via, stuff:Via, F.Cu at (138.2, 95.2)
- added REF**: Via, stuff:Via, F.Cu at (118.8, 85.2)
- added REF**: Via, stuff:Via, F.Cu at (138.2, 93.5)
- added REF**: Via, stuff:Via, F.Cu at (138.2, 98.5)
- added REF**: Via, stuff:Via, F.Cu at (138.2, 96.8)
- added REF**: Via, stuff:Via, F.Cu at (64.9, 81.3)
- added REF**: Via, stuff:Via, F.Cu at (63.6, 83.2)
- added REF**: Via, stuff:Via, F.Cu at (62.0, 84.0)
- added REF**: Via, stuff:Via, F.Cu at (61.0, 85.0)
- added REF**: Via, stuff:Via, F.Cu at (61.0, 87.0)
- added REF**: Via, stuff:Via, F.Cu at (61.0, 90.0)
- added REF**: Via, stuff:Via, F.Cu at (62.0, 92.0)
- added REF**: Via, stuff:Via, F.Cu at (113.8, 85.2)
- added REF**: Via, stuff:Via, F.Cu at (61.2, 95.2)
- added REF**: Via, stuff:Via, F.Cu at (58.8, 97.8)
- added REF**: Via, stuff:Via, F.Cu at (56.2, 95.2)
- added REF**: Via, stuff:Via, F.Cu at (53.8, 97.8)
- added REF**: Via, stuff:Via, F.Cu at (53.0, 93.0)
- added REF**: Via, stuff:Via, F.Cu at (52.0, 89.0)
- added REF**: Via, stuff:Via, F.Cu at (53.0, 85.0)
- added REF**: Via, stuff:Via, F.Cu at (52.0, 81.0)
- added REF**: Via, stuff:Via, F.Cu at (53.0, 77.0)
- added REF**: Via, stuff:Via, F.Cu at (52.0, 73.0)
- added REF**: Via, stuff:Via, F.Cu at (113.8, 82.8)
- added REF**: Via, stuff:Via, F.Cu at (53.0, 69.0)
- added REF**: Via, stuff:Via, F.Cu at (52.0, 65.0)
- added REF**: Via, stuff:Via, F.Cu at (53.0, 62.0)
- added REF**: Via, stuff:Via, F.Cu at (57.0, 62.0)
- added REF**: Via, stuff:Via, F.Cu at (61.0, 62.0)
- added REF**: Via, stuff:Via, F.Cu at (63.0, 59.0)
- added REF**: Via, stuff:Via, F.Cu at (65.0, 62.0)
- added REF**: Via, stuff:Via, F.Cu at (69.0, 62.0)
- added REF**: Via, stuff:Via, F.Cu at (67.0, 59.0)
- added REF**: Via, stuff:Via, F.Cu at (69.0, 57.0)
- added REF**: Via, stuff:Via, F.Cu at (108.8, 85.2)
- added REF**: Via, stuff:Via, F.Cu at (73.0, 59.0)
- added REF**: Via, stuff:Via, F.Cu at (76.0, 58.0)
- added REF**: Via, stuff:Via, F.Cu at (76.0, 55.0)
- added REF**: Via, stuff:Via, F.Cu at (73.0, 53.0)
- added REF**: Via, stuff:Via, F.Cu at (69.0, 53.0)
- added REF**: Via, stuff:Via, F.Cu at (108.8, 82.8)
- added REF**: Via, stuff:Via, F.Cu at (103.8, 82.8)
- added REF**: Via, stuff:Via, F.Cu at (103.8, 85.2)
- added REF**: Via, stuff:Via, F.Cu at (98.8, 85.2)
- added REF**: Via, stuff:Via, F.Cu at (121.2, 90.2)
- added REF**: Via, stuff:Via, F.Cu at (98.8, 82.8)
- added REF**: Via, stuff:Via, F.Cu at (93.8, 82.8)
- added REF**: Via, stuff:Via, F.Cu at (93.8, 85.2)
- added REF**: Via, stuff:Via, F.Cu at (88.8, 82.8)
- added REF**: Via, stuff:Via, F.Cu at (88.8, 85.2)
- added REF**: Via, stuff:Via, F.Cu at (62.0, 109.8)
- added REF**: Via, stuff:Via, F.Cu at (68.8, 109.8)
- added REF**: Via, stuff:Via, F.Cu at (68.8, 106.8)
- added REF**: Via, stuff:Via, F.Cu at (62.0, 106.8)
- added REF**: Via, stuff:Via, F.Cu at (52.2, 106.8)
- added REF**: Via, stuff:Via, F.Cu at (118.8, 100.2)
- added REF**: Via, stuff:Via, F.Cu at (56.0, 108.0)
- added REF**: Via, stuff:Via, F.Cu at (52.5, 110.8)
- added REF**: Via, stuff:Via, F.Cu at (58.0, 114.5)
- added REF**: Via, stuff:Via, F.Cu at (52.5, 114.2)
- added REF**: Via, stuff:Via, F.Cu at (66.2, 101.2)
- added REF**: Via, stuff:Via, F.Cu at (71.2, 101.2)
- added REF**: Via, stuff:Via, F.Cu at (73.8, 103.2)
- added REF**: Via, stuff:Via, F.Cu at (73.8, 105.2)
- added REF**: Via, stuff:Via, F.Cu at (73.8, 101.2)
- added REF**: Via, stuff:Via, F.Cu at (68.8, 101.2)
- added REF**: Via, stuff:Via, F.Cu at (118.8, 97.8)
- added REF**: Via, stuff:Via, F.Cu at (63.8, 101.2)
- added REF**: Via, stuff:Via, F.Cu at (61.2, 100.2)
- added REF**: Via, stuff:Via, F.Cu at (56.2, 100.2)
- added REF**: Via, stuff:Via, F.Cu at (51.2, 100.2)
- added REF**: Via, stuff:Via, F.Cu at (51.2, 95.2)
- added REF**: Via, stuff:Via, F.Cu at (61.2, 52.8)
- added REF**: Via, stuff:Via, F.Cu at (63.8, 52.8)
- added REF**: Via, stuff:Via, F.Cu at (63.8, 55.2)
- added REF**: Via, stuff:Via, F.Cu at (61.2, 55.2)
- added REF**: MountingHole_4.3mm_M4_Pad_Via, Mounting_Holes:MountingHole_4.3mm_M4_Pad_Via, F.Cu at (145.0, 145.0)
- added REF**: Via, stuff:Via, F.Cu at (118.8, 95.2)
- added REF**: MountingHole_4.3mm_M4_Pad_Via, Mounting_Holes:MountingHole_4.3mm_M4_Pad_Via, F.Cu at (55.0, 145.0)
- added REF**: MountingHole_4.3mm_M4_Pad_Via, Mounting_Holes:MountingHole_4.3mm_M4_Pad_Via, F.Cu at (55.0, 55.0)
- added REF**: Via, stuff:Via, F.Cu at (68.8, 148.6)
- added REF**: Via, stuff:Via, F.Cu at (71.2, 148.6)
- added REF**: Via, stuff:Via, F.Cu at (73.8, 148.6)
- added REF**: Via, stuff:Via, F.Cu at (76.2, 148.6)
- added REF**: Via, stuff:Via, F.Cu at (78.8, 148.6)
- added REF**: Via, stuff:Via, F.Cu at (83.8, 148.6)
- added REF**: MountingHole_4.3mm_M4_Pad_Via, Mounting_Holes:MountingHole_4.3mm_M4_Pad_Via, F.Cu at (145.0, 55.0)
- added REF**: Via, stuff:Via, F.Cu at (81.2, 148.6)
- added REF**: Via, stuff:Via, F.Cu at (86.2, 148.6)
- added REF**: Via, stuff:Via, F.Cu at (123.8, 90.2)
- added REF**: Via, stuff:Via, F.Cu at (88.8, 148.6)
- added REF**: Via, stuff:Via, F.Cu at (91.2, 148.6)
- added REF**: Via, stuff:Via, F.Cu at (93.8, 148.6)
- added REF**: Via, stuff:Via, F.Cu at (96.2, 148.6)
- added REF**: Via, stuff:Via, F.Cu at (98.8, 148.6)
- added REF**: Via, stuff:Via, F.Cu at (103.8, 148.6)
- added REF**: Via, stuff:Via, F.Cu at (101.2, 148.6)
- added REF**: Via, stuff:Via, F.Cu at (106.2, 148.6)
- added REF**: Via, stuff:Via, F.Cu at (108.8, 148.6)
- added REF**: Via, stuff:Via, F.Cu at (111.2, 148.6)
- added REF**: Via, stuff:Via, F.Cu at (123.8, 92.8)
- added REF**: Via, stuff:Via, F.Cu at (113.8, 148.6)
- added REF**: Via, stuff:Via, F.Cu at (116.2, 148.6)
- added REF**: Via, stuff:Via, F.Cu at (121.2, 148.6)
- added REF**: Via, stuff:Via, F.Cu at (118.8, 148.6)
- added REF**: Via, stuff:Via, F.Cu at (123.8, 148.6)
- added REF**: Via, stuff:Via, F.Cu at (126.2, 148.6)
- added REF**: Via, stuff:Via, F.Cu at (128.8, 148.6)
- added REF**: Via, stuff:Via, F.Cu at (131.2, 148.6)
- added REF**: Via, stuff:Via, F.Cu at (133.8, 148.6)
- added REF**: Via, stuff:Via, F.Cu at (136.2, 148.6)
- added REF**: Via, stuff:Via, F.Cu at (118.8, 92.8)
- added REF**: Via, stuff:Via, F.Cu at (138.8, 148.6)
- added REF**: Via, stuff:Via, F.Cu at (139.8, 106.2)
- added REF**: Via, stuff:Via, F.Cu at (143.6, 105.5)
- added REF**: Via, stuff:Via, F.Cu at (139.7, 110.5)
- added REF**: Via, stuff:Via, F.Cu at (143.8, 110.8)
- added REF**: Via, stuff:Via, F.Cu at (135.8, 115.0)
- added REF**: Via, stuff:Via, F.Cu at (135.7, 113.0)
- added REF**: Via, stuff:Via, F.Cu at (137.9, 113.8)
- added REF**: Via, stuff:Via, F.Cu at (142.8, 115.8)
- added REF**: Via, stuff:Via, F.Cu at (145.1, 116.0)
- added REF**: Via, stuff:Via, F.Cu at (118.8, 90.2)
- added REF**: Via, stuff:Via, F.Cu at (147.4, 116.0)
- added REF**: Via, stuff:Via, F.Cu at (128.7, 109.5)
- added REF**: Via, stuff:Via, F.Cu at (125.2, 109.3)
- added REF**: Via, stuff:Via, F.Cu at (125.2, 107.0)
- added REF**: Via, stuff:Via, F.Cu at (128.7, 107.0)
- added REF**: Via, stuff:Via, F.Cu at (128.8, 104.8)
- added REF**: Via, stuff:Via, F.Cu at (126.0, 104.7)
- added REF**: Via, stuff:Via, F.Cu at (129.3, 102.5)
- added REF**: Via, stuff:Via, F.Cu at (130.2, 100.2)
- added REF**: Via, stuff:Via, F.Cu at (130.1, 97.8)
- added U14: Si4435DY, Housings_SOIC:SOIC-8_3.9x4.9mm_Pitch1.27mm, B.Cu at (143.0, 98.0)
- added U15: DF12, stuff:DF12-20DP, F.Cu at (143.2, 87.8)
- added U16: LPC4370, stuff:BGA_100, F.Cu at (116.5, 57.0)
- added Y1: FK135EIHM0.032768, stuff:FK135, F.Cu at (129.0, 74.5)
- C25, R21, R22: moved to B.Cu
- moved C16 5.70 mm to (134.2, 143.5), turned to 270 degrees
- moved J6 4.47 mm to (132.5, 115.5)
- moved REF** 4.30 mm to (73.0, 57.0)
- moved C12 4.25 mm to (140.0, 124.0)
- moved REF** 2.93 mm to (142.0, 121.0)
- moved R22 1.77 mm to (124.8, 114.2), turned to 0 degrees
- moved J4 1.77 mm to (143.0, 118.0)
- moved C25 1.07 mm to (124.8, 116.2), turned to 180 degrees
- moved R21 0.63 mm to (128.5, 115.5)
- moved REF** 0.60 mm to (136.6, 145.7)
Connections:
- net /BAT_CHG/VIN renamed /VIN
- C40 pad 1: /BAT_CHG/SYS -> /DCDC_24V/PVIN
- C45 pad 2: /BAT_CHG/SYS -> /DCDC_24V/PVIN
- C47 pad 2: /BAT_CHG/SYS -> /DCDC_24V/PVIN
- C48 pad 2: /BAT_CHG/SYS -> /DCDC_24V/PVIN
- C51 pad 2: /BAT_CHG/SYS -> /DCDC_24V/PVIN
- C52 pad 2: /BAT_CHG/SYS -> /DCDC_24V/PVIN
- C53 pad 2: /BAT_CHG/SYS -> /DCDC_24V/PVIN
- J13 pad 1: /BAT_CHG/SYS -> /DCDC_24V/PVIN
- Q4 pad 2: /BAT_CHG/SYS -> /DCDC_24V/PVIN
- R57 pad 1: /BAT_CHG/SYS -> /DCDC_24V/PVIN
- R63 pad 1: /BAT_CHG/SYS -> /DCDC_24V/PVIN
- R65 pad 1: /BAT_CHG/SYS -> /DCDC_24V/PVIN
- R69 pad 1: /BAT_CHG/SYS -> /DCDC_24V/PVIN
- REF** pad 1: /BAT_CHG/SYS -> /DCDC_24V/PVIN
- U10 pad 2: /BAT_CHG/SYS -> /DCDC_24V/PVIN
- U10 pad 3: /BAT_CHG/SYS -> /DCDC_24V/PVIN
- U10 pad 4: /BAT_CHG/SYS -> /DCDC_24V/PVIN
- U13 pad 1: /BAT_CHG/SYS -> /DCDC_24V/PVIN
- U13 pad 2: /BAT_CHG/SYS -> /DCDC_24V/PVIN
- U13 pad 3: /BAT_CHG/SYS -> /DCDC_24V/PVIN
Routing:
- net /VIN: track 15.5 -> 71.4 mm
- net /DCDC_24V/PVIN: track 52.4 -> 96.4 mm, vias 0 -> 5
- net /BAT_CHG/SYS: track 42.0 -> 0.00 mm, vias 3 -> 0
- net GND: track 322.1 -> 361.0 mm, vias 53 -> 69
- net /VIN_PROT: track 0.00 -> 27.2 mm
- net /VIN_ADAPTER: track 0.00 -> 19.4 mm, vias 0 -> 3
- net /DCDC_24V/VOUT: track 25.2 -> 36.7 mm
- net /DCDC_24V/ISN: track 25.1 -> 30.0 mm, vias 2 -> 3
- net /DCDC_24V/ISP: track 67.0 -> 69.5 mm, vias 2 -> 1
- net Net-(D9-Pad2): track 0.00 -> 2.24 mm, vias 0 -> 1
- net Net-(F1-Pad2): track 0.00 -> 1.77 mm, vias 0 -> 1
- net /MCU_MAIN/VIO_3V3: track 0.00 -> 1.45 mm, vias 0 -> 1
- net (no net): track 0.00 -> 1.10 mm, vias 0 -> 1
- net /DCDC_24V/BST2: track 6.95 -> 7.85 mm
- added copper zone on B.Cu, net /DCDC_24V/PVIN
- added copper zone on F.Cu, net /DCDC_24V/PVIN
- added copper zone on VDDMix, net /MCU_MAIN/VIO_3V3
- added copper zone on B.Cu, net /VIN_PROT
- added copper zone on F.Cu, net /VIN_PROT
- added copper zone on B.Cu, net Net-(F1-Pad2)
- removed copper zone on B.Cu, net /BAT_CHG/SYS
- removed copper zone on F.Cu, net /BAT_CHG/SYS
Other:
- outline, holes or cut-outs redrawn
- net class Default: clearance 0.127 -> 0.1016; trace_width 0.127 -> 0.1016
- rule pad_to_mask_clearance: 0.127 -> 0.05
- rule trace_clearance: 0.127 -> 0.1016
- rule trace_min: 0.127 -> 0.1016
- rule via_min_drill: 0.3 -> 0.2
- rule via_min_size: 0.4 -> 0.45
- board text added: "Back"
- board text added: "Front"
- board text added: "Max. 4mm height in this section!"
