File: HamPWR.sch (KiCad schematic (older format))
At the start: 8 parts

Commit message: Progress
Parts:
- removed C?: 47µF 80V, Capacitors_SMD:CP_Elec_10x10.5, symbol CP
- removed C?: 220µF 35V, Capacitors_SMD:CP_Elec_8x10.5, symbol CP
- added C54, C55, C57: 10µF 100V, Capacitors_SMD:C_1210, symbol C
- added C58: 220µF 35V, Capacitors_SMD:CP_Elec_8x10.5, symbol CP
- added J14: PJ-082BH, stuff:pj-082bh, symbol Barrel_Jack
- added U15: DF12, stuff:DF12-20DP, symbol DF12
- C56: renamed from C?; Digikey (none) -> GMK325BJ106KN-T
- D9: renamed from D?; footprint Diodes_SMD:D_SMA -> Diodes_SMD:D_SOD-123
- F1: renamed from F?; value 10A Fast, 01020071Z -> 10A Fast, 0685H9100-01; footprint Fuse_Holders_and_Fuses:Fuseholder5x20_horiz_open_inline_Type-I -> Fuse_Holders_and_Fuses:Fuse_SMD1206_Reflow
- gave numbers to parts that had none: 3
Connections:
- net BAT_CHG/SYS: now also C58.1
- net GND: now also C54.2, C55.2, C57.2, C58.2, J14.2, J14.3
- net VIN: now also C57.1
- net VIN_ADAPTER: now also F1.1, J14.1; no longer U14.5 (D), U14.6 (D), U14.7 (D), U14.8 (D)
- net VIN_PROT: now also C54.1, C55.1
- net at F1.2: now also U14.5 (D), U14.6 (D), U14.7 (D), U14.8 (D)
Other:
- note added: "Pin 3 is shield\ninstead of switch"
Changed lines of the file:
@@
 LIBS:bq24765
 LIBS:mosfets
+LIBS:rjhse538x04
+LIBS:sm51589pel
+LIBS:df12
+LIBS:lpc4370
 LIBS:HamPWR-cache
 EELAYER 25 0
@@
 $Descr A4 11693 8268
 encoding utf-8
-Sheet 1 3
+Sheet 1 4
 Title ""
 Date ""
@@
 $EndSheet
 $Sheet
-S 4250 2700 1950 1400
+S 4700 2700 1950 1400
 U 5B036166
 F0 "BAT_CHG" 60
 F1 "BAT_CHG.sch" 60
-F2 "BAT" I R 6200 2850 60
-F3 "SYS" I L 4250 3200 60
-F4 "VICM" I R 6200 3100 60
-F5 "SDA" I R 6200 3200 60
-F6 "SCL" I R 6200 3300 60
-F7 "ACIN" I R 6200 3400 60
-F8 "ACOK" I R 6200 3500 60
-F9 "CE" I R 6200 3600 60
-F10 "ICOUT" I R 6200 3700 60
-F11 "/BYPASS" I R 6200 3800 60
-F12 "/ACDRV" I R 6200 3900 60
-F13 "/BATDRV" I L 4250 2850 60
-F14 "VIN" I L 4250 2950 60
+F2 "BAT" I R 6650 2850 60
+F3 "SYS" I L 4700 3200 60
+F4 "VICM" I R 6650 3100 60
+F5 "SDA" I R 6650 3200 60
+F6 "SCL" I R 6650 3300 60
+F7 "ACIN" I R 6650 3400 60
+F8 "ACOK" I R 6650 3500 60
+F9 "CE" I R 6650 3600 60
+F10 "ICOUT" I R 6650 3700 60
+F11 "/BYPASS" I R 6650 3800 60
+F12 "/ACDRV" I R 6650 3900 60
+F13 "/BATDRV" I L 4700 2850 60
+F14 "VIN" I L 4700 2950 60
 $EndSheet
 Wire Wire Line
-	4250 3200 3900 3200
+	3900 3200 4700 3200
 Wire Wire Line
 	3900 3200 3900 3300
@@
 	3900 3300 3600 3300
 $Comp
-L Si4435DY U?
+L Si4435DY U14
 U 1 1 5B041BA0
 P 1700 1300
-F 0 "U?" H 1700 1700 60  0000 C CNN
+F 0 "U14" H 1700 1700 60  0000 C CNN
 F 1 "Si4435DY" H 1700 1600 60  0000 C CNN
 F 2 "Housings_SOIC:SOIC-8_3.9x4.9mm_Pitch1.27mm" H 2650 1600 60  0001 C CNN
@@
 Wire Wire Line
 	2050 1150 2100 1150
-Wire Wire Line
-	2050 1250 2750 1250
 Wire Wire Line
 	2100 1350 2050 1350
@@
 VIN_PROT
 $Comp
-L R R?
+L R R71
 U 1 1 5B044B16
 P 1300 1700
-F 0 "R?" V 1380 1700 50  0000 C CNN
+F 0 "R71" V 1380 1700 50  0000 C CNN
 F 1 "10k" V 1300 1700 50  0000 C CNN
 F 2 "Resistors_SMD:R_0402" V 1230 1700 50  0001 C CNN
@@
 $EndComp
 $Comp
-L GND #PWR?
+L GND #PWR01
 U 1 1 5B044DC1
 P 1300 1900
-F 0 "#PWR?" H 1300 1650 50  0001 C CNN
+F 0 "#PWR01" H 1300 1650 50  0001 C CNN
 F 1 "GND" H 1300 1750 50  0000 C CNN
 F 2 "" H 1300 1900 50  0001 C CNN
@@
 	1250 1450 1350 1450
 $Comp
-L D_Zener D?
+L D_Zener D9
 U 1 1 5B044FD7
 P 1100 1450
-F 0 "D?" H 1100 1550 50  0000 C CNN
+F 0 "D9" H 1100 1550 50  0000 C CNN
 F 1 "10V" H 1100 1350 50  0000 C CNN
-F 2 "Diodes_SMD:D_SMA" H 1100 1450 50  0001 C CNN
+F 2 "Diodes_SMD:D_SOD-123" H 1100 1450 50  0001 C CNN
 F 3 "" H 1100 1450 50  0001 C CNN
 	1    1100 1450
@@
 	2100 1150 2100 1450
 $Comp
-L Fuse F?
+L Fuse F1
 U 1 1 5B04846C
 P 2450 1250
-F 0 "F?" V 2530 1250 50  0000 C CNN
-F 1 "10A Fast, 01020071Z" V 2650 1500 50  0000 C CNN
-F 2 "Fuse_Holders_and_Fuses:Fuseholder5x20_horiz_open_inline_Type-I" V 2380 1250 50  0001 C CNN
+F 0 "F1" V 2530 1250 50  0000 C CNN
+F 1 "10A Fast, 0685H9100-01" V 2650 1500 50  0000 C CNN
+F 2 "Fuse_Holders_and_Fuses:Fuse_SMD1206_Reflow" V 2380 1250 50  0001 C CNN
 F 3 "" H 2450 1250 50  0001 C CNN
 	1    2450 1250
@@
 $EndComp
 $Comp
-L L_Core_Ferrite L?
+L L_Core_Ferrite L3
 U 1 1 5B0491D4
 P 4850 1100
-F 0 "L?" V 4800 1100 50  0000 C CNN
+F 0 "L3" V 4800 1100 50  0000 C CNN
 F 1 "SRP1265A-5R6M" V 4960 1100 50  0000 C CNN
 F 2 "stuff:SRP1265A" H 4850 1100 50  0001 C CNN
@@
 Adapter filter
 $Comp
-L CP C?
-U 1 1 5B04EEFE
-P 4350 1350
-F 0 "C?" H 4375 1450 50  0000 L CNN
-F 1 "47µF 80V" V 4450 900 50  0000 L CNN
-F 2 "Capacitors_SMD:CP_Elec_10x10.5" H 4388 1200 50  0001 C CNN
-F 3 "" H 4350 1350 50  0001 C CNN
-F 4 "https://www.digikey.at/product-detail/de/panasonic-electronic-components/EEE-TG1K470UP/PCE4107CT-ND/817778" H 4350 1350 60  0001 C CNN "Digikey"
-	1    4350 1350
-	1    0    0    -1
-$EndComp
-$Comp
-L CP C?
-U 1 1 5B0508BA
-P 5250 1350
-F 0 "C?" H 5275 1450 50  0000 L CNN
-F 1 "220µF 35V" V 5350 850 50  0000 L CNN
-F 2 "Capacitors_SMD:CP_Elec_8x10.5" H 5288 1200 50  0001 C CNN
-F 3 "" H 5250 1350 50  0001 C CNN
-F 4 "https://www.digikey.at/product-detail/de/panasonic-electronic-components/EEE-FT1H221AP/PCE5025CT-ND/2652080" H 5250 1350 60  0001 C CNN "Digikey"
-	1    5250 1350
-	1    0    0    -1
-$EndComp
-$Comp
-L C C?
+L C C56
 U 1 1 5B05176C
 P 5550 1350
-F 0 "C?" H 5575 1450 50  0000 L CNN
+F 0 "C56" H 5575 1450 50  0000 L CNN
 F 1 "10µF 100V" V 5650 850 50  0000 L CNN
 F 2 "Capacitors_SMD:C_1210" H 5588 1200 50  0001 C CNN
 F 3 "" H 5550 1350 50  0001 C CNN
+F 4 "GMK325BJ106KN-T" H 5550 1350 60  0001 C CNN "Digikey"
 	1    5550 1350
 	1    0    0    -1
 $EndComp
 $Comp
-L GND #PWR?
+L GND #PWR02
 U 1 1 5B05200A
 P 4350 1550
-F 0 "#PWR?" H 4350 1300 50  0001 C CNN
+F 0 "#PWR02" H 4350 1300 50  0001 C CNN
 F 1 "GND" H 4350 1400 50  0000 C CNN
 F 2 "" H 4350 1550 50  0001 C CNN
@@
 $EndComp
 $Comp
-L GND #PWR?
+L GND #PWR03
 U 1 1 5B0520CA
 P 5250 1550
-F 0 "#PWR?" H 5250 1300 50  0001 C CNN
+F 0 "#PWR03" H 5250 1300 50  0001 C CNN
 F 1 "GND" H 5250 1400 50  0000 C CNN
 F 2 "" H 5250 1550 50  0001 C CNN
@@
 $EndComp
 $Comp
-L GND #PWR?
+L GND #PWR04
 U 1 1 5B052183
 P 5550 1550
-F 0 "#PWR?" H 5550 1300 50  0001 C CNN
+F 0 "#PWR04" H 5550 1300 50  0001 C CNN
 F 1 "GND" H 5550 1400 50  0000 C CNN
 F 2 "" H 5550 1550 50  0001 C CNN
@@
 	5550 1100 5550 1200
 Connection ~ 5250 1100
+Connection ~ 5550 1100
+Text Label 4600 2950 2    60   ~ 0
+VIN
+Wire Wire Line
+	4600 2950 4700 2950
+Text Notes 2250 1050 0    60   ~ 0
+Fuse cap\n3527C\nKeystone Electronics
+$Comp
+L Barrel_Jack J14
+U 1 1 5B057429
+P 7250 1200
+F 0 "J14" H 7250 1410 50  0000 C CNN
+F 1 "PJ-082BH" H 7250 1025 50  0000 C CNN
+F 2 "stuff:pj-082bh" H 7300 1160 50  0001 C CNN
+F 3 "" H 7300 1160 50  0001 C CNN
+	1    7250 1200
+	-1   0    0    1
+$EndComp
+Text Notes 6850 900  0    60   ~ 0
+Pin 3 is shield\ninstead of switch
+Wire Wire Line
+	6950 1200 6850 1200
+Wire Wire Line
+	6850 1200 6850 1100
+Wire Wire Line
+	6800 1100 6950 1100
 Text Label 5700 1100 0    60   ~ 0
 VIN
-Connection ~ 5550 1100
-Text Label 4150 2950 2    60   ~ 0
-VIN
-Wire Wire Line
-	4150 2950 4250 2950
-Text Notes 2250 1050 0    60   ~ 0
-Fuse cap\n3527C\nKeystone Electronics
+Text Label 6750 1300 2    60   ~ 0
+VIN_ADAPTER
+Wire Wire Line
+	6750 1300 6950 1300
+$Comp
+L GND #PWR05
+U 1 1 5B0589A5
+P 6800 1100
+F 0 "#PWR05" H 6800 850 50  0001 C CNN
+F 1 "GND" H 6800 950 50  0000 C CNN
+F 2 "" H 6800 1100 50  0001 C CNN
+F 3 "" H 6800 1100 50  0001 C CNN
+	1    6800 1100
+	0    1    1    0
+$EndComp
+Connection ~ 6850 1100
+$Comp
+L DF12 U15
+U 1 1 5B05B3F7
+P 9350 2600
+F 0 "U15" H 9500 2600 60  0000 C CNN
+F 1 "DF12" H 9200 2600 60  0000 C CNN
+F 2 "stuff:DF12-20DP" H 9350 2600 60  0001 C CNN
+F 3 "" H 9350 2600 60  0001 C CNN
+	1    9350 2600
+	0    1    1    0
+$EndComp
+Wire Wire Line
+	2050 1250 2300 1250
+Wire Wire Line
+	2600 1250 2750 1250
+$Comp
+L C C57
+U 1 1 5B061A6A
+P 5250 1350
+F 0 "C57" H 5275 1450 50  0000 L CNN
+F 1 "10µF 100V" V 5350 850 50  0000 L CNN
+F 2 "Capacitors_SMD:C_1210" H 5288 1200 50  0001 C CNN
+F 3 "" H 5250 1350 50  0001 C CNN
+F 4 "GMK325BJ106KN-T" H 5250 1350 60  0001 C CNN "Digikey"
+	1    5250 1350
+	1    0    0    -1
+$EndComp
+$Comp
+L GND #PWR06
+U 1 1 5B061D54
+P 4600 1550
+F 0 "#PWR06" H 4600 1300 50  0001 C CNN
+F 1 "GND" H 4600 1400 50  0000 C CNN
+F 2 "" H 4600 1550 50  0001 C CNN
+F 3 "" H 4600 1550 50  0001 C CNN
+	1    4600 1550
+	1    0    0    -1
+$EndComp
+Wire Wire Line
+	4600 1550 4600 1500
+Wire Wire Line
+	4600 1200 4600 1100
+Connection ~ 4600 1100
+$Comp
+L C C55
+U 1 1 5B06225A
+P 4600 1350
+F 0 "C55" H 4625 1450 50  0000 L CNN
+F 1 "10µF 100V" V 4700 850 50  0000 L CNN
+F 2 "Capacitors_SMD:C_1210" H 4638 1200 50  0001 C CNN
+F 3 "" H 4600 1350 50  0001 C CNN
+F 4 "GMK325BJ106KN-T" H 4600 1350 60  0001 C CNN "Digikey"
+	1    4600 1350
+	1    0    0    -1
+$EndComp
+$Comp
+L C C54
+U 1 1 5B06233E
+P 4350 1350
+F 0 "C54" H 4375 1450 50  0000 L CNN
+F 1 "10µF 100V" V 4450 850 50  0000 L CNN
+F 2 "Capacitors_SMD:C_1210" H 4388 1200 50  0001 C CNN
+F 3 "" H 4350 1350 50  0001 C CNN
+F 4 "GMK325BJ106KN-T" H 4350 1350 60  0001 C CNN "Digikey"
+	1    4350 1350
+	1    0    0    -1
+$EndComp
+$Comp
+L CP C58
+U 1 1 5B0645E9
+P 4100 3400
+F 0 "C58" H 4125 3500 50  0000 L CNN
+F 1 "220µF 35V" V 4100 3700 50  0000 L CNN
+F 2 "Capacitors_SMD:CP_Elec_8x10.5" H 4138 3250 50  0001 C CNN
+F 3 "" H 4100 3400 50  0001 C CNN
+F 4 "https://www.digikey.at/product-detail/de/panasonic-electronic-components/EEE-FT1H221AP/PCE5025CT-ND/2652080" H 4100 3400 60  0001 C CNN "Digikey"
+	1    4100 3400
+	1    0    0    -1
+$EndComp
+Wire Wire Line
+	4100 3550 4100 3600
+Wire Wire Line
+	4100 3250 4100 3200
+Connection ~ 4100 3200
+$Comp
+L GND #PWR07
+U 1 1 5B06473B
+P 4100 3600
+F 0 "#PWR07" H 4100 3350 50  0001 C CNN
+F 1 "GND" H 4100 3450 50  0000 C CNN
+F 2 "" H 4100 3600 50  0001 C CNN
+F 3 "" H 4100 3600 50  0001 C CNN
+	1    4100 3600
+	1    0    0    -1
+$EndComp
+$Sheet
+S 1600 4500 2000 1300
+U 5B065DB3
+F0 "MCU_MAIN" 60
+F1 "MCU_MAIN.sch" 60
+$EndSheet
 $EndSCHEMATC
